Commit message: not calibrated urdf

File: rsm/urdf/colorado.urdf (robot description, URDF)
Before this commit: robot colorado, 3 links, 2 joints
Links:
- added link cam1_link; visual box size=0.05 0.05 0.05
- added link cam2_link; visual box size=0.05 0.05 0.05
Joints:
- removed joint base_to_nav
- added joint cam1_to_cam2: type fixed, parent cam1_link, child cam2_link, origin xyz=0.6 0 0
- added joint velodyne_to_cam1: type fixed, parent velodyne_link, child cam1_link, origin xyz=0.21 0.3 -0.2 rpy=-1.5707 0 -1.5707
- added joint velodyne_to_nav: type fixed, parent velodyne_link, child nav_link, origin xyz=-0.3 -0.25 -0.1
- joint base_to_velodyne: origin xyz=2.5 0 2.0 -> xyz=2.0 0 2.0

Commit message: updating the mask processing bridge
the bridge is realy not ready a lot of things to do but it it incapsulate the integrations ideas from the mitting with sasha

File: rsm/urdf/colorado.urdf (robot description, URDF)
Before this commit: robot colorado, 5 links, 4 joints
Joints:
- joint base_to_velodyne: origin xyz=2.0 0 2.0 -> xyz=1.0 0 2.0
- joint cam1_to_cam2: origin xyz=0.6 0 0 -> xyz=0 -0.6 0
- joint velodyne_to_cam1: origin xyz=0.21 0.3 -0.2 rpy=-1.5707 0 -1.5707 -> xyz=0.21 0.3 -0.2 rpy=0 0 0

Commit message: change in colorado urdf

File: rsm/urdf/colorado.urdf (robot description, URDF)
Before this commit: robot colorado, 5 links, 4 joints
Joints:
- joint velodyne_to_nav: origin xyz=-0.3 -0.25 -0.1 -> xyz=-1.0 -0.25 -0.1
